File: estopsupport.kicad_sch (KiCad schematic)
At the start: 23 parts, among them J1 ESTOP1, J2 ESTOP2, J3 CONTACTOR, J4 TAP_ESTOP, J5 5V_IN, J6 PWR, U1 PC817, U2 BTS6163D

Commit message: fix: shunt resistor value changed to datasheet recommendation
Parts:
- R4: value 10k -> 1k
Other:
- note added: "Sense resistor for measuring Isense Non-automated but simpler Nominal Isense is about 0.33 mA Fault Isense is >5 mA"
- note removed: "Shunt for measuring fault Non-automated but simpler Nominal Isense is about 0.33 mA Fault Isense is >5 mA"
Changed lines of the file:
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@@
 		(comment 2 "Designed to operate a Kilovac using 2 5V switches in series")
 	)
-	(text "Shunt for measuring fault\nNon-automated but simpler\nNominal Isense is about 0.33 mA\nFault Isense is >5 mA"
+	(text "Sense resistor for measuring Isense\nNon-automated but simpler\nNominal Isense is about 0.33 mA\nFault Isense is >5 mA"
 		(exclude_from_sim no)
 		(at 81.026 71.628 0)
@@
 			)
 		)
-		(property "Value" "10k"
+		(property "Value" "1k"
 			(at 85.09 74.9299 0)
 			(show_name no)

Commit message: feat: started BOM, added ground lines to tap
Parts:
- C1: JLCPCB Part # (none) -> C48543040
- C2: JLCPCB Part # (none) -> C24497
- D1: JLCPCB Part # (none) -> C16015
- D2: JLCPCB Part # (none) -> C2909831
- J4: footprint Connector_PinSocket_2.54mm:PinSocket_1x04_P2.54mm_Horizontal -> Connector_PinSocket_2.54mm:PinSocket_2x04_P2.54mm_Horizontal; symbol Connector:Conn_01x04_Pin -> Connector_Generic:Conn_02x04_Odd_Even
- R2: value 6.2k -> 1.6k
- U1: JLCPCB Part # (none) -> C5350
- U2: JLCPCB Part # (none) -> C534821
Connections:
- net GNDD: now also J4.2 (Pin_2), J4.4 (Pin_4), J4.6 (Pin_6), J4.8 (Pin_8)
- net at J4.1 (Pin_1), J4.3 (Pin_3), R5.2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: now also J4.5 (Pin_5), J4.7 (Pin_7); no longer J4.2 (Pin_2), J4.4 (Pin_4)

Commit message: feat: change to use battery voltage directly for powering the coil
Parts:
- added D4: SMCJ22A, Diode_SMD:D_SMC, symbol Device:D_Zener
- added F1: Fuse, Fuse:Fuse_1206_3216Metric_Pad1.42x1.75mm_HandSolder, symbol Device:Fuse
- C1: value 100u -> 22u; footprint Capacitor_SMD:CP_Elec_6.3x7.7 -> Capacitor_SMD:CP_Elec_4x5.4
- R5: value 3.3k -> 4.3k
Connections:
- net +12V: no longer C1.1, C2.1, J6.1 (Pin_1), U2.3 (Vbb)
- net GND: now also D4.2 (A)
- new net: F1.1, U2.3 (Vbb)
- new net +BATT: C1.1, C2.1, D4.1 (K), F1.2, J6.1 (Pin_1)
Other:
- note added: "Expected: 4S battery 12-16.8V"
- moved on the sheet: C1, C2
