File: estopsupport.kicad_pcb (KiCad board)
At the start: 2 copper layers, 60 x 35 mm, 26 parts, among them J1 PWR, J2 CONTACTOR, J3 ESTOP2, J4 ESTOP1, J5 TAP_ESTOP, J6 5V_IN, U1 PC817, U2 BTS6163D

Commit message: final adjustments for ordering
Parts:
- added REF**: ToolingHole_1.152mm, MountingHole:ToolingHole_1.152mm, F.Cu at (71.5, 62.8)
- added REF**: ToolingHole_1.152mm, MountingHole:ToolingHole_1.152mm, F.Cu at (93.0, 33.3)
- D3, F1: moved to F.Cu
- moved REF** 23.2 mm to (37.0, 33.3)
- moved D2 11.9 mm to (77.7, 62.3), turned to 0 degrees
- moved R6 10.5 mm to (83.5, 62.3)
- moved F1 9.01 mm to (74.0, 45.3)
- moved D3 6.96 mm to (67.0, 46.3), turned to 180 degrees
- moved C2 6.73 mm to (75.5, 52.3), turned to -135 degrees
- moved R3 5.59 mm to (49.0, 51.8), turned to -90 degrees
- moved C1 5.15 mm to (82.0, 48.3), turned to 135 degrees
- moved U1 3.89 mm to (53.0, 42.3)
- moved U2 3.61 mm to (84.5, 54.3), turned to -135 degrees
- moved R5 3.35 mm to (51.0, 49.3)
- moved R4 2.55 mm to (90.0, 48.6)
- moved G*** 2.24 mm to (66.5, 60.8)
- moved R2 2.24 mm to (53.5, 39.8)
- moved D1 2.00 mm to (50.0, 44.3)
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Routing:
- net Net-(D2-K): track 11.3 -> 28.6 mm
- net +BATT: track 16.1 -> 0.00 mm, vias 6 -> 0
- net Net-(J1-Pin_1): track 4.46 -> 8.34 mm
- net GNDD: track 11.7 -> 14.2 mm
- net GND: track 10.2 -> 12.4 mm
- net Net-(U2-IN): track 18.4 -> 16.6 mm
- net Net-(J5-Pin_1): track 12.9 -> 14.7 mm
- net Net-(D1-K): track 4.55 -> 3.07 mm
- net Net-(D1-A): track 8.46 -> 9.53 mm
- net Net-(J2-Pin_1): track 21.5 -> 20.6 mm
- net Net-(R2-Pad2): track 3.85 -> 3.05 mm
- net Net-(U2-IS): track 3.91 -> 3.29 mm
Other:
- board text added: "-"
- board text added: "S"

Commit message: minor fixes and updates
Parts:
- removed J2: CONTACTOR, TerminalBlock_Phoenix:TerminalBlock_Phoenix_MKDS-1,5-2_1x02_P5.00mm_Horizontal
- removed the REF** at (93.0, 33.3)
- added D4: 1N4007, Diode_SMD:D_SMA, F.Cu at (81.5, 70.8)
- added D5: MM1W24, Diode_SMD:D_SOD-123, F.Cu at (72.8, 70.8)
- added K1: Relay_SPST-NO, EasyEDA_Lib:RELAY-TH_JQX-V7H-012-1HP, F.Cu at (105.1, 72.3)
- added Q1: PN2222A, Package_TO_SOT_THT:TO-92_Inline, F.Cu at (61.2, 72.1)
- added R7: 15, Resistor_SMD:R_1812_4532Metric, F.Cu at (115.9, 56.3)
- added R8: 1k, Resistor_SMD:R_0603_1608Metric, F.Cu at (68.2, 76.3)
- J1: value PWR -> Barrier Block 1x3; footprint TerminalBlock_Phoenix:TerminalBlock_Phoenix_MKDS-1,5-2_1x02_P5.00mm_Horizontal -> EasyEDA_Lib:CONN-TH_KF88SA-16.0-3P
- J3: value ESTOP2 -> Dupont 1x2
- J4: value ESTOP1 -> Dupont 1x2
- J5: value TAP_ESTOP -> Dupont 2x4
- J6: value 5V_IN -> Dupont 1x2
- moved J1 68.1 mm to (133.5, 61.8), turned to -90 degrees
- moved H4 65.1 mm to (149.0, 88.8)
- moved H2 58.6 mm to (148.5, 33.3)
- moved U2 34.2 mm to (115.7, 40.4), turned to 45 degrees
- moved D3 32.2 mm to (98.6, 40.3)
- moved J5 31.9 mm to (73.2, 76.6)
- moved J6 29.1 mm to (64.5, 79.3)
- moved H3 27.7 mm to (36.5, 88.8)
- moved R6 27.3 mm to (105.7, 46.3)
- moved F1 27.2 mm to (99.5, 54.8), turned to 0 degrees
- moved R4 25.6 mm to (115.5, 50.8), turned to 180 degrees
- moved R3 25.3 mm to (56.5, 76.0)
- moved U1 24.8 mm to (74.4, 54.8)
- moved R2 21.0 mm to (69.2, 53.8)
- moved R5 21.0 mm to (66.7, 63.3)
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Connections:
- F1 pad 1: Net-(J1-Pin_1) -> Net-(U2-Vbb)
- J1 pad 1: Net-(J1-Pin_1) -> +BATT
- R3 pad 1: Net-(J5-Pin_1) -> Net-(Q1-B)
- R5 pad 2: Net-(J5-Pin_1) -> Net-(Q1-B)
- U2 pad 3: +BATT -> Net-(U2-Vbb)
Routing:
- net Net-(D4-K): track 20.6 -> 0.00 mm
- net GND: track 12.4 -> 30.1 mm
- net Net-(D2-A): track 2.41 -> 19.0 mm
- net Net-(U2-IN): track 16.6 -> 0.00 mm
- net Net-(Q1-B): track 0.00 -> 14.7 mm
- net Net-(J5-Pin_1): track 14.7 -> 0.00 mm
- net Net-(D1-A): track 9.53 -> 21.3 mm
- net GNDD: track 14.2 -> 2.50 mm
- net Net-(R2-Pad2): track 3.05 -> 9.29 mm
- net Net-(U2-IS): track 3.29 -> 0.00 mm
Other:
- board size 60 x 35 mm -> 2 x 2 mm
- board text added: "GND 5V TAP"
- board text removed: "5V GNDD TAP"
